File: BSPD/BSPD.kicad_sch (KiCad schematic)
At the start: 32 parts, among them Q3 PMOS, U1 LM339DR, U10 641964-1, U2 SN74LVC1G08DBVR, U3 NE555DR, U4 SN74LVC3G14DCUR, U5 SN74AC32DR, U6 SN74LVC1G08DBVR, U7 641964-1, U8 R-78E5.0-0.5, U9 641964-1

Commit message: Layout
Connections:
- net 10%_THROTTLE: now also U1.10 (4IN-); no longer U1.8 (3IN-)
- net BSE_IN: now also U1.9 (3IN+); no longer U1.11 (4IN+)
- net GND: no longer R4.1, U4.6 (3A)
- net HARD_BREAK: now also U1.8 (3IN-); no longer U1.10 (4IN-)
- net THROTTLE_IN: now also U1.11 (4IN+); no longer U1.9 (3IN+)
- new net: R4.1, U4.6 (3A)
- no-connect marks 1 -> 3
Other:
- moved on the sheet: R4
Changed lines of the file:
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@@
 	)
 	(junction
-		(at 234.95 195.58)
-		(diameter 0)
-		(color 0 0 0 0)
-	)
-	(junction
 		(at 323.85 205.74)
 		(diameter 0)
@@
 	)
 	(no_connect
+		(at 166.37 234.95)
+	)
+	(no_connect
 		(at 375.92 233.68)
 	)
+	(no_connect
+		(at 222.25 237.49)
+	)
 	(wire
 		(pts
-			(xy 245.11 170.18) (xy 245.11 168.91)
+			(xy 222.25 195.58) (xy 220.98 195.58)
 		)
 		(stroke
@@
 	(wire
 		(pts
-			(xy 222.25 224.79) (xy 224.79 224.79)
+			(xy 245.11 170.18) (xy 245.11 168.91)
 		)
 		(stroke
@@
 	(wire
 		(pts
-			(xy 220.98 195.58) (xy 234.95 195.58)
+			(xy 222.25 224.79) (xy 224.79 224.79)
 		)
 		(stroke
@@
 	(wire
 		(pts
-			(xy 299.72 27.94) (xy 302.26 27.94)
+			(xy 180.34 115.57) (xy 187.96 115.57)
 		)
 		(stroke
@@
 	(wire
 		(pts
-			(xy 115.57 154.94) (xy 115.57 146.05)
+			(xy 299.72 27.94) (xy 302.26 27.94)
 		)
 		(stroke
@@
 	(wire
 		(pts
-			(xy 229.87 165.1) (xy 231.14 165.1)
+			(xy 115.57 154.94) (xy 115.57 146.05)
 		)
 		(stroke
@@
 	(wire
 		(pts
-			(xy 299.72 38.1) (xy 299.72 41.91)
+			(xy 229.87 165.1) (xy 231.14 165.1)
 		)
 		(stroke
@@
 	(wire
 		(pts
-			(xy 220.98 191.77) (xy 220.98 187.96)
+			(xy 299.72 38.1) (xy 299.72 41.91)
 		)
 		(stroke
@@
 	(wire
 		(pts
-			(xy 111.76 120.65) (xy 119.38 120.65)
+			(xy 220.98 191.77) (xy 220.98 187.96)
 		)
 		(stroke
@@
 	(wire
 		(pts
-			(xy 260.35 231.14) (xy 260.35 229.87)
+			(xy 111.76 120.65) (xy 119.38 120.65)
 		)
 		(stroke
@@
 	(wire
 		(pts
-			(xy 199.39 115.57) (xy 180.34 115.57)
+			(xy 260.35 231.14) (xy 260.35 229.87)
 		)
 		(stroke
@@
 	(wire
 		(pts
+			(xy 189.23 120.65) (xy 184.15 120.65)
+		)
+		(stroke
+			(width 0)
+			(type default)
+		)
+	)
+	(wire
+		(pts
 			(xy 273.05 219.71) (xy 302.26 219.71)
 		)
@@
 	(wire
 		(pts
+			(xy 222.25 201.93) (xy 222.25 195.58)
+		)
+		(stroke
+			(width 0)
+			(type default)
+		)
+	)
+	(wire
+		(pts
 			(xy 309.88 217.17) (xy 309.88 215.9)
 		)
@@
 	(wire
 		(pts
+			(xy 180.34 120.65) (xy 180.34 127)
+		)
+		(stroke
+			(width 0)
+			(type default)
+		)
+	)
+	(wire
+		(pts
 			(xy 189.23 39.37) (xy 189.23 43.18)
 		)
@@
 	(wire
 		(pts
+			(xy 238.76 195.58) (xy 238.76 201.93)
+		)
+		(stroke
+			(width 0)
+			(type default)
+		)
+	)
+	(wire
+		(pts
 			(xy 231.14 236.22) (xy 226.06 236.22)
 		)
@@
 	(wire
 		(pts
+			(xy 184.15 120.65) (xy 184.15 118.11)
+		)
+		(stroke
+			(width 0)
+			(type default)
+		)
+	)
+	(wire
+		(pts
 			(xy 92.71 24.13) (xy 92.71 26.67)
 		)
@@
 	(wire
 		(pts
+			(xy 180.34 127) (xy 201.93 127)
+		)
+		(stroke
+			(width 0)
+			(type default)
+		)
+	)
+	(wire
+		(pts
 			(xy 260.35 201.93) (xy 278.13 201.93)
 		)
@@
 	(wire
 		(pts
+			(xy 189.23 124.46) (xy 189.23 120.65)
+		)
+		(stroke
+			(width 0)
+			(type default)
+		)
+	)
+	(wire
+		(pts
 			(xy 231.14 162.56) (xy 231.14 163.83)
 		)
@@
 	(wire
 		(pts
+			(xy 243.84 195.58) (xy 238.76 195.58)
+		)
+		(stroke
+			(width 0)
+			(type default)
+		)
+	)
+	(wire
+		(pts
 			(xy 302.26 219.71) (xy 302.26 200.66)
 		)
@@
 	(wire
 		(pts
-			(xy 199.39 120.65) (xy 180.34 120.65)
+			(xy 158.75 232.41) (xy 158.75 231.14)
 		)
 		(stroke
@@
 	(wire
 		(pts
-			(xy 158.75 232.41) (xy 158.75 231.14)
+			(xy 226.06 210.82) (xy 165.1 210.82)
 		)
 		(stroke
@@
 	(wire
 		(pts
-			(xy 226.06 210.82) (xy 165.1 210.82)
+			(xy 163.83 187.96) (xy 163.83 194.31)
 		)
 		(stroke
@@
 	(wire
 		(pts
-			(xy 163.83 187.96) (xy 163.83 194.31)
+			(xy 323.85 187.96) (xy 323.85 205.74)
 		)
 		(stroke
@@
 	(wire
 		(pts
-			(xy 323.85 187.96) (xy 323.85 205.74)
+			(xy 226.06 194.31) (xy 226.06 210.82)
 		)
 		(stroke
@@
 	(wire
 		(pts
-			(xy 226.06 194.31) (xy 226.06 210.82)
+			(xy 238.76 201.93) (xy 222.25 201.93)
 		)
 		(stroke
@@
 	(wire
 		(pts
+			(xy 184.15 118.11) (xy 180.34 118.11)
+		)
+		(stroke
+			(width 0)
+			(type default)
+		)
+	)
+	(wire
+		(pts
 			(xy 166.37 229.87) (xy 166.37 231.14)
 		)
@@
 	(wire
 		(pts
-			(xy 243.84 195.58) (xy 243.84 196.85)
+			(xy 243.84 195.58) (xy 243.84 198.12)
 		)
 		(stroke
@@
 	(wire
 		(pts
-			(xy 234.95 195.58) (xy 243.84 195.58)
+			(xy 87.63 26.67) (xy 92.71 26.67)
 		)
 		(stroke
@@
 	(wire
 		(pts
-			(xy 87.63 26.67) (xy 92.71 26.67)
+			(xy 222.25 232.41) (xy 222.25 233.68)
 		)
 		(stroke
@@
 	(wire
 		(pts
-			(xy 222.25 232.41) (xy 222.25 233.68)
+			(xy 180.34 113.03) (xy 185.42 113.03)
 		)
 		(stroke
@@
 	(global_label "10%_THROTTLE"
 		(shape input)
-		(at 199.39 120.65 0)
+		(at 187.96 115.57 0)
 		(fields_autoplaced yes)
 		(effects
@@
 		)
 		(property "Intersheetrefs" "${INTERSHEET_REFS}"
-			(at 216.2241 120.65 0)
+			(at 204.7941 115.57 0)
 			(effects
 				(font
@@
 	(global_label "HARD_BREAK"
 		(shape input)
-		(at 199.39 115.57 0)
+		(at 201.93 127 0)
 		(fields_autoplaced yes)
 		(effects
@@
 		)
 		(property "Intersheetrefs" "${INTERSHEET_REFS}"
-			(at 214.3495 115.57 0)
+			(at 216.8895 127 0)
 			(effects
 				(font
@@
 	(global_label "THROTTLE_IN"
 		(shape input)
-		(at 180.34 118.11 0)
+		(at 185.42 113.03 0)
 		(fields_autoplaced yes)
 		(effects
@@
 		)
 		(property "Intersheetrefs" "${INTERSHEET_REFS}"
-			(at 195.239 118.11 0)
+			(at 200.319 113.03 0)
 			(effects
 				(font
@@
 	(global_label "BSE_IN"
 		(shape input)
-		(at 180.34 113.03 0)
+		(at 189.23 124.46 0)
 		(fields_autoplaced yes)
 		(effects
@@
 		)
 		(property "Intersheetrefs" "${INTERSHEET_REFS}"
-			(at 189.8566 113.03 0)
+			(at 198.7466 124.46 0)
 			(effects
 				(font
@@
 	(symbol
 		(lib_id "power:GND")
-		(at 243.84 204.47 0)
+		(at 243.84 205.74 0)
 		(unit 1)
 		(exclude_from_sim no)
@@
 		(fields_autoplaced yes)
 		(property "Reference" "#PWR024"
-			(at 243.84 210.82 0)
+			(at 243.84 212.09 0)
 			(effects
 				(font
@@
 		)
 		(property "Value" "GND"
-			(at 243.84 209.55 0)
+			(at 243.84 210.82 0)
 			(effects
 				(font
@@
 		)
 		(property "Footprint" ""
-			(at 243.84 204.47 0)
+			(at 243.84 205.74 0)
 			(effects
 				(font
@@
 		)
 		(property "Datasheet" ""
-			(at 243.84 204.47 0)
+			(at 243.84 205.74 0)
 			(effects
 				(font
@@
 		)
 		(property "Description" "Power symbol creates a global label with name \"GND\" , ground"
-			(at 243.84 204.47 0)
+			(at 243.84 205.74 0)
 			(effects
 				(font
@@
 	(symbol
 		(lib_id "Device:R_US")
-		(at 243.84 200.66 0)
+		(at 243.84 201.93 0)
 		(unit 1)
 		(exclude_from_sim no)
@@
 		(fields_autoplaced yes)
 		(property "Reference" "R4"
-			(at 246.38 199.3899 0)
+			(at 246.38 200.6599 0)
 			(effects
 				(font
@@
 		)
 		(property "Value" "10K"
-			(at 246.38 201.9299 0)
+			(at 246.38 203.1999 0)
 			(effects
 				(font
@@
 		)
 		(property "Footprint" "Resistor_SMD:R_0805_2012Metric"
-			(at 244.856 200.914 90)
+			(at 244.856 202.184 90)
 			(effects
 				(font
@@
 		)
 		(property "Datasheet" "~"
-			(at 243.84 200.66 0)
+			(at 243.84 201.93 0)
 			(effects
 				(font
@@
 		)
 		(property "Description" "Resistor, US symbol"
-			(at 243.84 200.66 0)
+			(at 243.84 201.93 0)
 			(effects
 				(font

Commit message: JLC PCB BOM, placement redone to account for footprint changes, started re-routing
Parts:
- C1, C10, C2: JLCPCB Part # (none) -> C1713
- C11: footprint Capacitor_SMD:C_0805_2012Metric -> Capacitor_SMD:C_0402_1005Metric; JLCPCB Part # (none) -> C1524
- C12, C13, C14, C3, C9: footprint Capacitor_SMD:C_0805_2012Metric -> Capacitor_SMD:C_0402_1005Metric; JLCPCB Part # (none) -> C1525
- R1: footprint Resistor_SMD:R_0402_1005Metric -> Resistor_SMD:R_1206_3216Metric; JLCPCB Part # (none) -> C102061
- R2, R3, R4: footprint Resistor_SMD:R_0805_2012Metric -> Resistor_SMD:R_1206_3216Metric; JLCPCB Part # (none) -> C1489
- RV1, RV2, RV3, RV4: footprint PVG3A103C01R00:RES_C01R00 -> 3224W-1-103E:POT_3224W; JLCPCB Part # (none) -> C81348
- U1: JLCPCB Part # (none) -> C7948
- U10, U7, U9: now not fitted
- U2: footprint SN74LVC1G08DBVR:DBV0005A_N -> SN74LVC1G08DBVR:DBV0005A_L; JLCPCB Part # (none) -> C7666
- U3: JLCPCB Part # (none) -> C7593
- U4: JLCPCB Part # (none) -> C98856
- U5: JLCPCB Part # (none) -> C352943
- U6: JLCPCB Part # (none) -> C7666
- U8: JLCPCB Part # (none) -> C18212367
