File: Fault Latch/Fault Latch 2/Fault Latch 2.kicad_sch (KiCad schematic)
At the start: 111 parts, among them K101 Fujitsu_FTR-LYAA005x, K102 Fujitsu_FTR-LYAA005x, K103 Fujitsu_FTR-LYAA005x, Q102 Q_NMOS_GSD, Q104 Q_NPN_BEC, Q106 Q_NPN_BEC, Q107 Q_NPN_BEC, Q108 Q_NPN_BEC, Q109 Q_NMOS_GDS, Q110 Q_NMOS_GDS, Q111 Q_NMOS_GDS, Q112 Q_NPN_BEC, Q113 Q_NPN_BEC, Q114 Q_NMOS_GDS, Q115 Q_NMOS_GSD, Q116 Q_NMOS_GSD, Q117 Q_NMOS_GDS, Q118 Q_NMOS_GDS, Q119 Q_NMOS_GDS, SW101 SW_Omron_B3FS, SW102 SW_Omron_B3FS, SW103 SW_Omron_B3FS, U101 641964-1, U102 74AHC1G00, U103 74AHC1G00, U104 74AHC1G00, U105 641964-1, U106 74LS279, U110 641964-1, U111 641964-1, U112 641964-1, U113 641964-1, U114 SFH617A-1, U115 SFH617A-1, U116 SFH617A-1, U118 LM555xM, U119 641964-1, U120 74AHC1G08, U121 641964-1, U122 641964-1, U123 SFH617A-1, U125 SFH617A-1, U126 SFH617A-1

Commit message: Almost complete merge of fault latch and tssi, footprint still not working for PMOS
Parts:
- removed D104: D_Schottky, Diode_SMD:D_SMA, symbol Device:D_Schottky
- removed K101: Fujitsu_FTR-LYAA005x, Relay_THT:Relay_SPST-NO_Fujitsu_FTR-LYAA005x_FormA_Vertical, symbol Relay:Fujitsu_FTR-LYAA005x
- removed Q109, Q110, Q118, Q119: Q_NMOS_GDS, Package_TO_SOT_SMD:TO-252-2, symbol Transistor_FET:Q_NMOS_GDS
- removed U110: 641964-1, 641964-1:TE_641964-1, symbol CONNECTOR:641964-1
- removed U123: SFH617A-1, Package_DIP:DIP-4_W7.62mm, symbol Isolator:SFH617A-1
- added D109: D_Schottky, Diode_SMD:D_SMA, symbol Device:D_Schottky
- added K104: Fujitsu_FTR-LYAA005x, Relay_THT:Relay_SPST-NO_Fujitsu_FTR-LYAA005x_FormA_Vertical, symbol Relay:Fujitsu_FTR-LYAA005x
- added Q105, Q109, Q110, Q118: Q_PMOS_GSD, Package_TO_SOT_SMD:SOT-523, symbol Transistor_FET:Q_PMOS_GSD
- added U117: 641964-1, 641964-1:TE_641964-1, symbol CONNECTOR:641964-1
- added U127: SFH617A-1, Package_DIP:DIP-4_W7.62mm, symbol Isolator:SFH617A-1
Connections:
- net +5V: now also Q105.3 (D), Q109.3 (D), Q110.3 (D), Q118.3 (D); no longer R141.1, R142.1, U125.1
- net BMS_Green: no longer Q117.2 (D), R140.2
- net BMS_SR: now also D109.1 (K), K104.A1, Q110.1 (G), U127.2
- net GND: now also D105.2 (A), K102.A2, R141.2, R142.2, D109.2 (A), K104.A2
- net GNDPWR: now also U127.3
- net IMD_Green: now also Q117.2 (D), R140.2
- net IMD_SR: now also D105.1 (K), K102.A1, U125.2, Q118.1 (G); no longer D105.2 (A), K102.A2
- net at Q117.1 (G), R138.2: now also U127.4
- net at D3.2 (A): now also R141.1, Q110.2 (S); no longer R141.2
- net at D4.2 (A): now also R142.1, Q118.2 (S); no longer R142.2
- net at D103.1 (K), U106.4 (Q): now also Q109.1 (G)
- net at D107.1 (K), U106.7 (Q): now also Q105.1 (G)
- new net: Q105.2 (S), U125.1
- new net: K104.13, U117.1
- new net: K104.14, U117.2
- new net: Q109.2 (S), U127.1
Other:
- moved on the sheet: C102, C103, C104, C107, C108, C109, C110, C111, C113, C114, C115, C116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
