File: RML/RML.kicad_pcb (KiCad board)
At the start: 4 copper layers, 85 x 50 mm, 29 parts, among them Q101 Q_NMOS_GDS, Q102 Q_NMOS_GDS, U101 641964-1, U102 LM555xM, U103 SFH617A-1, U104 74AHC1G02, U105 641964-1, U106 641964-1, U107 LM7805_TO220

Commit message: Fault Latch V2.0 waiting for final check
Routing:
- net +5V: track 32.9 -> 43.7 mm
Changed lines of the file:
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@@
+	)
+	(segment
+		(start 109 59.96586)
+		(end 106.34 62.62586)
+		(width 0.5)
+		(layer "F.Cu")
+		(net 4)
 	)
 	(segment
@@
 		(width 0.5)
 		(layer "F.Cu")
+		(net 4)
+	)
+	(segment
+		(start 109 53)
+		(end 109 59.96586)
+		(width 0.5)
+		(layer "F.Cu")

Commit message: RML READY
Routing:
- net GND: track 7.95 -> 0.20 mm, vias 8 -> 206
- net +5V: track 43.7 -> 47.3 mm
- net GNDPWR: vias 0 -> 101
- added copper zone on F.Cu, net GNDPWR
- removed copper zone on F.Cu, net +5V
