File: glr-2024e-fault-latch.kicad_sch (KiCad schematic)
At the start: 67 parts, among them K101 Fujitsu_FTR-LYAA005x, K103 Fujitsu_FTR-LYAA005x, Q101 Q_NPN_BEC, Q102 Q_NPN_BEC, Q103 Q_NPN_BEC, Q104 Q_NPN_BEC, Q105 Q_NMOS_GSD, Q106 Q_NMOS_GSD, Q107 Q_PMOS_GSD, Q108 Q_PMOS_GSD, Q114 Q_NMOS_GSD, Q115 Q_NMOS_GSD, SW101 SW_Omron_B3FS, SW102 SW_Omron_B3FS, U101 SFH617A-1, U102 SFH617A-1, U104 74AHC1G00, U105 74AHC1G00, U107 74LS279, U108 641964-1, U109 SFH617A-1, U110 SFH617A-1, U112 641964-1, U115 641964-1, U116 641964-1, U120 641964-1, U123 641964-1

Commit message: use to screw terminals
improve labels in schematic

Co-Authored-By: wallalex0 <97884125+wallalex0@users.noreply.github.com>
Parts:
- removed U108, U112, U115, U116, U120, U123: 641964-1, 641964-1:TE_641964-1, symbol CONNECTOR:641964-1
- added J1: Screw_Terminal_01x08, GLR_KiCad_Library:WECO-950-FB-08, symbol Connector:Screw_Terminal_01x08
- added J2: Screw_Terminal_01x04, GLR_KiCad_Library:WECO-950-FB-04, symbol Connector:Screw_Terminal_01x04
Connections:
- net +12V: now also J1.2 (Pin_2)
- net BMS_INPUT: now also J1.8 (Pin_8)
- net GNDPWR: now also J1.1 (Pin_1)
- net IMD_INPUT: now also J1.7 (Pin_7)
- net IMD_LED_12V: now reaches R112.2
- net IMD_LED_12V: now also J1.4 (Pin_4)
- net IMD_LED_GND: now reaches Q106.3 (D)
- net IMD_LED_GND: now also J1.3 (Pin_3)
- net BMS_LED_GND: now reaches Q115.3 (D)
- net BMS_LED_GND: now also J1.5 (Pin_5)
- net BMS_LED_12V: now reaches R135.2
- net BMS_LED_12V: now also J1.6 (Pin_6)
- net BMS_GREEN renamed BMS_LED
- net BMS_SR: no longer names the net of D102.1 (K), Q107.1 (G), U107.4 (Q)
- net IMD_SR: no longer names the net of D101.1 (K), Q108.1 (G), U107.7 (Q)
- net NRESET_BMS renamed BMS_NRESET
- net SDC renamed BMS_SDC_IN
- net BMS_SDC_IN: now also J2.3 (Pin_3); no longer K103.14
- net SDC_IN renamed IMD_SDC_IN
- net IMD_SDC_IN: now also J2.1 (Pin_1)
- net SDC_OUT renamed BMS_SDC_OUT
- net BMS_SDC_OUT: now also J2.4 (Pin_4)
- new net IMD_SDC_OUT: J2.2 (Pin_2), K103.14
- no-connect marks 9 -> 7
Other:
- note removed: "12V"
- moved on the sheet: C102, D102, R109, R112, R117, R121, R135, R136, U104, U107A
